File: pcb/MCU.kicad_sch (KiCad schematic)
At the start: 36 parts, among them J2 Tag connect TC2030-CTX, SW1 RESET, U1 nRF52840, Y1 32MHz, Y2 32.768kHz

Commit message: buck converter and updates
Parts:
- removed D1: RED, LED_SMD:LED_0603_1608Metric, symbol Device:LED
- removed D2: YELLOW, LED_SMD:LED_0603_1608Metric, symbol Device:LED
- removed R1, R2: 680, Resistor_SMD:R_0603_1608Metric, symbol Device:R_Small
- C11: now fitted; now in the parts list

Commit message: switch TCXO, laid out from ref design from nordic
Parts:
- C15, C16, C21: footprint Capacitor_SMD:C_0805_2012Metric -> Capacitor_SMD:C_0603_1608Metric
- L2, L3: footprint Inductor_SMD:L_0805_2012Metric -> Inductor_SMD:L_0603_1608Metric
Changed lines of the file:
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@@
 			)
 		)
-		(property "Footprint" "Capacitor_SMD:C_0805_2012Metric"
+		(property "Footprint" "Capacitor_SMD:C_0603_1608Metric"
 			(at 203.2 119.38 0)
 			(hide yes)
@@
 			)
 		)
-		(property "Footprint" "Capacitor_SMD:C_0805_2012Metric"
+		(property "Footprint" "Capacitor_SMD:C_0603_1608Metric"
 			(at 179.07 148.59 0)
 			(hide yes)
@@
 			)
 		)
-		(property "Footprint" "Inductor_SMD:L_0805_2012Metric"
+		(property "Footprint" "Inductor_SMD:L_0603_1608Metric"
 			(at 116.84 27.94 0)
 			(hide yes)
@@
 			)
 		)
-		(property "Footprint" "Inductor_SMD:L_0805_2012Metric"
+		(property "Footprint" "Inductor_SMD:L_0603_1608Metric"
 			(at 121.92 31.75 0)
 			(hide yes)
@@
 			)
 		)
-		(property "Footprint" "Capacitor_SMD:C_0805_2012Metric"
+		(property "Footprint" "Capacitor_SMD:C_0603_1608Metric"
 			(at 217.17 128.27 0)
 			(hide yes)

Commit message: V2
Parts:
- removed J2: Tag connect TC2030-CTX, Connector_PinHeader_2.54mm:PinHeader_2x03_P2.54mm_Vertical, symbol Connector_Generic:Conn_02x03_Counter_Clockwise
- added TP10, TP11, TP8, TP9: TestPoint, TestPoint:TestPoint_Pad_D1.0mm, symbol Connector:TestPoint
- TP3: renamed from TP12; footprint TestPoint:TestPoint_Pad_2.0x2.0mm -> TestPoint:TestPoint_Pad_D1.0mm
- TP4: renamed from TP11; footprint TestPoint:TestPoint_Pad_2.0x2.0mm -> TestPoint:TestPoint_Pad_D1.0mm
- renumbered C6 to C1, C9 to C10, C17 to C11, C10 to C12, C21 to C13, C11 to C14, C18 to C15, C12 to C16, C19 to C17, C13 to C18, C14 to C19, C7 to C2, C15 to C21, C1 to C3, C2 to C4, C3 to C6, C4 to C7, C16 to C9, L2 to L1, L4 to L2, L1 to L4, Y2 to Y1, Y1 to Y2
Connections:
- net RX_LED is gone; now on net ANT_SW: U1.N1 (P0.08)
- net TX_LED is gone; now on net BT_MODE: U1.L1 (P0.06)
- net ANT_SW: no longer U1.B19 (P1.11)
- net BT_MODE: no longer U1.AD8 (P0.13)
- net BT_PDN: now also U1.J24 (NFC2/P0.10); no longer U1.L24 (NFC1/P0.09)
- net BT_RX_EN: now also U1.A10 (AIN5/P0.29); no longer U1.AD18 (P0.22)
- net BT_TX_EN: now also U1.A12 (AIN0/P0.02); no longer U1.AD20 (P0.24)
- net LORA_BUSY: now also U1.L24 (NFC1/P0.09); no longer U1.A10 (AIN5/P0.29)
- net LORA_CS: now also U1.AD8 (P0.13); no longer U1.AD10 (P0.15)
- net LORA_MISO: now also U1.AD10 (P0.15); no longer U1.A14 (P1.15)
- net LORA_MOSI: now also U1.AD18 (P0.22); no longer U1.A16 (P1.13)
- net LORA_NRST: now also U1.J1 (AIN2/P0.04); no longer U1.A12 (AIN0/P0.02)
- net LORA_SCK: now also U1.AD20 (P0.24); no longer U1.A20 (P1.10)
- net NRST: now also TP11.1
- net SWDCLK: now also TP9.1
- net SWDIO: now also TP10.1
- net SWO: now also TP8.1
- net UART_RX: now also U1.R1 (TRACEDATA3/P1.09); no longer U1.G1 (P0.26)
- net UART_TX: now also U1.U1 (TRACEDATA1/P0.12); no longer U1.J1 (AIN2/P0.04)
- new net I2C1_SCL: U1.A14 (P1.15)
- new net I2C1_SDA: U1.G1 (P0.26)
- new net I2C2_SCL: U1.A20 (P1.10)
- new net I2C2_SDA: U1.A16 (P1.13)
- no-connect marks 22 -> 20
Other:
- note added: "Avoid use of "NFC" and "AIN" pins for signals over 10kHz. Pins are located near RF Blocks and could crosstalk with 2.4GHz signal"
- note removed: "Doesn't have to be tag connect footprint"
- title: (none) -> nRF52840 Interface MCU

Commit message: fix SWD position
Parts:
- added TP12: TestPoint, TestPoint:TestPoint_Pad_D1.0mm, symbol Connector:TestPoint
Connections:
- net GND: now also TP12.1
Changed lines of the file:
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@@
 	(rectangle
 		(start 224.79 109.22)
-		(end 269.24 138.43)
+		(end 273.05 138.43)
 		(stroke
 			(width 0)
@@
 	(wire
 		(pts
+			(xy 255.27 116.84) (xy 256.54 116.84)
+		)
+		(stroke
+			(width 0)
+			(type default)
+		)
+	)
+	(wire
+		(pts
 			(xy 68.58 104.14) (xy 62.23 104.14)
 		)
@@
 	)
 	(symbol
+		(lib_id "Connector:TestPoint")
+		(at 256.54 116.84 270)
+		(unit 1)
+		(body_style 1)
+		(exclude_from_sim no)
+		(in_bom yes)
+		(on_board yes)
+		(in_pos_files yes)
+		(dnp no)
+		(fields_autoplaced yes)
+		(property "Reference" "TP12"
+			(at 261.62 115.5699 90)
+			(show_name no)
+			(do_not_autoplace no)
+			(effects
+				(font
+					(size 1.27 1.27)
+				)
+				(justify left)
+			)
+		)
+		(property "Value" "TestPoint"
+			(at 261.62 118.1099 90)
+			(show_name no)
+			(do_not_autoplace no)
+			(effects
+				(font
+					(size 1.27 1.27)
+				)
+				(justify left)
+			)
+		)
+		(property "Footprint" "TestPoint:TestPoint_Pad_D1.0mm"
+			(at 256.54 121.92 0)
+			(hide yes)
+			(show_name no)
+			(do_not_autoplace no)
+			(effects
+				(font
+					(size 1.27 1.27)
+				)
+			)
+		)
+		(property "Datasheet" ""
+			(at 256.54 121.92 0)
+			(hide yes)
+			(show_name no)
+			(do_not_autoplace no)
+			(effects
+				(font
+					(size 1.27 1.27)
+				)
+			)
+		)
+		(property "Description" "test point"
+			(at 256.54 116.84 0)
+			(hide yes)
+			(show_name no)
+			(do_not_autoplace no)
+			(effects
+				(font
+					(size 1.27 1.27)
+				)
+			)
+		)
+		(property "KLC_S3.3" ""
+			(at 256.54 116.84 90)
+			(hide yes)
+			(show_name no)
+			(do_not_autoplace no)
+			(effects
+				(font
+					(size 1.27 1.27)
+				)
+			)
+		)
+		(property "KLC_S4.1" ""
+			(at 256.54 116.84 90)
+			(hide yes)
+			(show_name no)
+			(do_not_autoplace no)
+			(effects
+				(font
+					(size 1.27 1.27)
+				)
+			)
+		)
+		(pin "1"
+		)
+		(instances
+			(project "pcb"
+				(path "/52b1b5de-c493-4cfe-b90b-d072cb2fb98d/c650ee69-dc51-4c07-96ce-be5227ce12c9"
+					(reference "TP12")
+					(unit 1)
+				)
+			)
+		)
+	)
+	(symbol
 		(lib_id "Device:C_Small")
 		(at 156.21 38.1 90)
@@
 					(unit 1)
 				)
+			)
+		)
+	)
+	(symbol
+		(lib_id "power:GND")
+		(at 255.27 116.84 0)
+		(unit 1)
+		(body_style 1)
+		(exclude_from_sim no)
+		(in_bom yes)
+		(on_board yes)
+		(in_pos_files yes)
+		(dnp no)
+		(fields_autoplaced yes)
+		(property "Reference" "#PWR024"
+			(at 255.27 123.19 0)
+			(hide yes)
+			(show_name no)
+			(do_not_autoplace no)
+			(effects
+				(font
+					(size 1.27 1.27)
+				)
+			)
+		)
+		(property "Value" "GND"
+			(at 255.27 121.92 0)
+			(show_name no)
+			(do_not_autoplace no)
+			(effects
+				(font
+					(size 1.27 1.27)
+				)
+			)
+		)
+		(property "Footprint" ""
+			(at 255.27 116.84 0)
+			(hide yes)
+			(show_name no)
+			(do_not_autoplace no)
+			(effects
+				(font
+					(size 1.27 1.27)
+				)
+			)
+		)
+		(property "Datasheet" ""
+			(at 255.27 116.84 0)
+			(hide yes)
+			(show_name no)
+			(do_not_autoplace no)
+			(effects
+				(font
+					(size 1.27 1.27)
+				)
+			)
+		)
+		(property "Description" "Power symbol creates a global label with name \"GND\" , ground"
+			(at 255.27 116.84 0)
+			(hide yes)
+			(show_name no)
+			(do_not_autoplace no)
+			(effects
+				(font
+					(size 1.27 1.27)
+				)
+			)
+		)
+		(pin "1"
+		)
+		(instances
+			(project "pcb"
+				(path "/52b1b5de-c493-4cfe-b90b-d072cb2fb98d/c650ee69-dc51-4c07-96ce-be5227ce12c9"
+					(reference "#PWR024")
+					(unit 1)
+				)

Commit message: revision 3
Parts:
- removed C10, C19: DNP, Capacitor_SMD:C_0402_1005Metric, symbol Device:C_Small
- removed L3: 10uH, Inductor_SMD:L_0603_1608Metric, symbol Device:L_Small
- removed TP10, TP11, TP12, TP9: TestPoint, TestPoint:TestPoint_Pad_D1.0mm, symbol Connector:TestPoint
- removed TP3: VDD (nRF regulated), TestPoint:TestPoint_Pad_D1.0mm, symbol Connector:TestPoint
- added J7: SWD Breakout, Connector_PinHeader_2.54mm:PinHeader_2x03_P2.54mm_Vertical, symbol Connector_Generic:Conn_02x03_Counter_Clockwise
- TP8: value TestPoint -> DCC
Connections:
- net VDD is gone; now on net +3.3V: C11.1, C15.1, C17.1, C20.1, U1.A22 (VDD), U1.AD14 (VDD), U1.AD23 (VDD), U1.B1 (VDD), U1.W1 (VDD)
- net +3.3V: now also J7.6 (Pin_6)
- net DCC: now also TP8.1
- net GND: now also J7.4 (Pin_4)
- net NRST: now also J7.5 (Pin_5)
- net SWDCLK: now also J7.2 (Pin_2)
- net SWDIO: now also J7.3 (Pin_3)
- net SWO: now also J7.1 (Pin_1); no longer TP8.1
- no-connect marks 20 -> 25
Other:
- note added: "Config 5 No Internal Regulator, VDD and VDDH supplied from the onboard 3.3V LDO"
- note removed: "VDD is chip regulated 3v3 with an internal LDO Don't supply VDD from an external source"
