File: pcb/USB.kicad_sch (KiCad schematic)
At the start: 4 parts, among them J3 USB C 2.0 Receptacle, U2 USBLC6-2SC6

Commit message: V2
Parts:
- renumbered J3 to J8, R3 to R1, R4 to R2
Changed lines of the file:
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@@
 		(dnp no)
 		(fields_autoplaced yes)
-		(property "Reference" "#PWR021"
+		(property "Reference" "#PWR037"
 			(at 128.27 113.03 0)
 			(hide yes)
@@
 			(project "pcb"
 				(path "/52b1b5de-c493-4cfe-b90b-d072cb2fb98d/ed5a3bba-7415-47bc-8e5e-36238a3b783c"
-					(reference "#PWR021")
+					(reference "#PWR037")
 					(unit 1)
 				)
@@
 		(in_pos_files yes)
 		(dnp no)
-		(property "Reference" "R4"
+		(property "Reference" "R2"
 			(at 149.606 92.456 90)
 			(show_name no)
@@
 			(project "pcb"
 				(path "/52b1b5de-c493-4cfe-b90b-d072cb2fb98d/ed5a3bba-7415-47bc-8e5e-36238a3b783c"
-					(reference "R4")
+					(reference "R2")
 					(unit 1)
 				)
@@
 		(dnp no)
 		(fields_autoplaced yes)
-		(property "Reference" "#PWR023"
+		(property "Reference" "#PWR034"
 			(at 152.4 83.82 0)
 			(hide yes)
@@
 			(project "pcb"
 				(path "/52b1b5de-c493-4cfe-b90b-d072cb2fb98d/ed5a3bba-7415-47bc-8e5e-36238a3b783c"
-					(reference "#PWR023")
+					(reference "#PWR034")
 					(unit 1)
 				)
@@
 		(in_pos_files yes)
 		(dnp no)
-		(property "Reference" "R3"
+		(property "Reference" "R1"
 			(at 149.352 85.344 90)
 			(show_name no)
@@
 			(project "pcb"
 				(path "/52b1b5de-c493-4cfe-b90b-d072cb2fb98d/ed5a3bba-7415-47bc-8e5e-36238a3b783c"
-					(reference "R3")
+					(reference "R1")
 					(unit 1)
 				)
@@
 		(dnp no)
 		(fields_autoplaced yes)
-		(property "Reference" "#PWR057"
+		(property "Reference" "#PWR033"
 			(at 243.84 44.45 0)
 			(hide yes)
@@
 			(project "pcb"
 				(path "/52b1b5de-c493-4cfe-b90b-d072cb2fb98d/ed5a3bba-7415-47bc-8e5e-36238a3b783c"
-					(reference "#PWR057")
+					(reference "#PWR033")
 					(unit 1)
 				)
@@
 		(dnp no)
 		(fields_autoplaced yes)
-		(property "Reference" "#PWR024"
+		(property "Reference" "#PWR038"
 			(at 176.53 129.54 0)
 			(hide yes)
@@
 			(project "pcb"
 				(path "/52b1b5de-c493-4cfe-b90b-d072cb2fb98d/ed5a3bba-7415-47bc-8e5e-36238a3b783c"
-					(reference "#PWR024")
+					(reference "#PWR038")
 					(unit 1)
 				)
@@
 		(dnp no)
 		(fields_autoplaced yes)
-		(property "Reference" "#PWR022"
+		(property "Reference" "#PWR035"
 			(at 146.05 96.52 0)
 			(hide yes)
@@
 			(project "pcb"
 				(path "/52b1b5de-c493-4cfe-b90b-d072cb2fb98d/ed5a3bba-7415-47bc-8e5e-36238a3b783c"
-					(reference "#PWR022")
+					(reference "#PWR035")
 					(unit 1)
 				)
@@
 		(in_pos_files yes)
 		(dnp no)
-		(property "Reference" "J3"
+		(property "Reference" "J8"
 			(at 172.72 74.93 0)
 			(show_name no)
@@
 			(project "pcb"
 				(path "/52b1b5de-c493-4cfe-b90b-d072cb2fb98d/ed5a3bba-7415-47bc-8e5e-36238a3b783c"
-					(reference "J3")
+					(reference "J8")
 					(unit 1)
 				)
@@
 		(in_pos_files yes)
 		(dnp no)
-		(property "Reference" "#PWR020"
+		(property "Reference" "#PWR036"
 			(at 128.27 95.25 0)
 			(hide yes)
@@
 			(project "pcb"
 				(path "/52b1b5de-c493-4cfe-b90b-d072cb2fb98d/ed5a3bba-7415-47bc-8e5e-36238a3b783c"
-					(reference "#PWR020")
-					(unit 1)
-				)
+					(reference "#PWR036")
+					(unit 1)
+				)
