File: pcb/bluetooth.kicad_sch (KiCad schematic)
At the start: 12 parts, among them U4 nRF21540

Commit message: buck converter and updates
Changed lines of the file:
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@@
+		)
+	)
+	(label "BT_DEC"
+		(at 116.84 67.31 0)
+		(effects
+			(font
+				(size 1.27 1.27)
+			)
+			(justify left bottom)
 		)
 	)

Commit message: V2
Parts:
- C36: renamed from C26; footprint Capacitor_SMD:C_0805_2012Metric -> Capacitor_SMD:C_0603_1608Metric
- renumbered C25 to C35, C27 to C37, C28 to C38, C24 to C39, L5 to L6, L6 to L7, R7 to R11, R6 to R12, R8 to R13, U4 to U5
Changed lines of the file:
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@@
 		(in_pos_files yes)
 		(dnp no)
-		(property "Reference" "#PWR032"
+		(property "Reference" "#PWR056"
 			(at 115.57 69.85 0)
 			(hide yes)
@@
 			(project "pcb"
 				(path "/52b1b5de-c493-4cfe-b90b-d072cb2fb98d/9ecc0d26-f5db-4725-b97a-75ab22334c44"
-					(reference "#PWR032")
+					(reference "#PWR056")
 					(unit 1)
 				)
@@
 		(in_pos_files yes)
 		(dnp no)
-		(property "Reference" "C26"
+		(property "Reference" "C36"
 			(at 123.19 69.8562 0)
 			(show_name no)
@@
 			)
 		)
-		(property "Footprint" "Capacitor_SMD:C_0805_2012Metric"
+		(property "Footprint" "Capacitor_SMD:C_0603_1608Metric"
 			(at 125.73 71.12 0)
 			(hide yes)
@@
 			(project "pcb"
 				(path "/52b1b5de-c493-4cfe-b90b-d072cb2fb98d/9ecc0d26-f5db-4725-b97a-75ab22334c44"
-					(reference "C26")
+					(reference "C36")
 					(unit 1)
 				)
@@
 		(dnp no)
 		(fields_autoplaced yes)
-		(property "Reference" "R8"
+		(property "Reference" "R13"
 			(at 153.67 114.2999 0)
 			(show_name no)
@@
 			(project "pcb"
 				(path "/52b1b5de-c493-4cfe-b90b-d072cb2fb98d/9ecc0d26-f5db-4725-b97a-75ab22334c44"
-					(reference "R8")
+					(reference "R13")
 					(unit 1)
 				)
@@
 		(dnp no)
 		(fields_autoplaced yes)
-		(property "Reference" "#PWR033"
+		(property "Reference" "#PWR057"
 			(at 115.57 82.55 0)
 			(hide yes)
@@
 			(project "pcb"
 				(path "/52b1b5de-c493-4cfe-b90b-d072cb2fb98d/9ecc0d26-f5db-4725-b97a-75ab22334c44"
-					(reference "#PWR033")
+					(reference "#PWR057")
 					(unit 1)
 				)
@@
 		(dnp no)
 		(fields_autoplaced yes)
-		(property "Reference" "L6"
+		(property "Reference" "L7"
 			(at 170.18 91.44 90)
 			(show_name no)
@@
 			(project "pcb"
 				(path "/52b1b5de-c493-4cfe-b90b-d072cb2fb98d/9ecc0d26-f5db-4725-b97a-75ab22334c44"
-					(reference "L6")
+					(reference "L7")
 					(unit 1)
 				)
@@
 		(dnp no)
 		(fields_autoplaced yes)
-		(property "Reference" "#PWR035"
+		(property "Reference" "#PWR062"
 			(at 130.81 132.08 0)
 			(hide yes)
@@
 			(project "pcb"
 				(path "/52b1b5de-c493-4cfe-b90b-d072cb2fb98d/9ecc0d26-f5db-4725-b97a-75ab22334c44"
-					(reference "#PWR035")
+					(reference "#PWR062")
 					(unit 1)
 				)
@@
 		(dnp no)
 		(fields_autoplaced yes)
-		(property "Reference" "#PWR038"
+		(property "Reference" "#PWR054"
 			(at 243.84 35.56 0)
 			(hide yes)
@@
 			(project "pcb"
 				(path "/52b1b5de-c493-4cfe-b90b-d072cb2fb98d/9ecc0d26-f5db-4725-b97a-75ab22334c44"
-					(reference "#PWR038")
+					(reference "#PWR054")
 					(unit 1)
 				)
@@
 		(dnp no)
 		(fields_autoplaced yes)
-		(property "Reference" "U4"
+		(property "Reference" "U5"
 			(at 140.97 81.534 0)
 			(show_name no)
@@
 			(project "pcb"
 				(path "/52b1b5de-c493-4cfe-b90b-d072cb2fb98d/9ecc0d26-f5db-4725-b97a-75ab22334c44"
-					(reference "U4")
+					(reference "U5")
 					(unit 1)
 				)
@@
 		(in_pos_files yes)
 		(dnp no)
-		(property "Reference" "C27"
+		(property "Reference" "C37"
 			(at 161.29 99.0662 0)
 			(show_name no)
@@
 			(project "pcb"
 				(path "/52b1b5de-c493-4cfe-b90b-d072cb2fb98d/9ecc0d26-f5db-4725-b97a-75ab22334c44"
-					(reference "C27")
+					(reference "C37")
 					(unit 1)
 				)
@@
 		(dnp no)
 		(fields_autoplaced yes)
-		(property "Reference" "#PWR037"
+		(property "Reference" "#PWR059"
 			(at 185.42 109.22 0)
 			(hide yes)
@@
 			(project "pcb"
 				(path "/52b1b5de-c493-4cfe-b90b-d072cb2fb98d/9ecc0d26-f5db-4725-b97a-75ab22334c44"
-					(reference "#PWR037")
+					(reference "#PWR059")
 					(unit 1)
 				)
@@
 		(dnp no)
 		(fields_autoplaced yes)
-		(property "Reference" "#PWR036"
+		(property "Reference" "#PWR060"
 			(at 176.53 111.76 0)
 			(hide yes)
@@
 			(project "pcb"
 				(path "/52b1b5de-c493-4cfe-b90b-d072cb2fb98d/9ecc0d26-f5db-4725-b97a-75ab22334c44"
-					(reference "#PWR036")
+					(reference "#PWR060")
 					(unit 1)
 				)
@@
 		(dnp no)
 		(fields_autoplaced yes)
-		(property "Reference" "L5"
+		(property "Reference" "L6"
 			(at 157.48 91.44 90)
 			(show_name no)
@@
 			(project "pcb"
 				(path "/52b1b5de-c493-4cfe-b90b-d072cb2fb98d/9ecc0d26-f5db-4725-b97a-75ab22334c44"
-					(reference "L5")
+					(reference "L6")
 					(unit 1)
 				)
@@
 		(in_pos_files yes)
 		(dnp no)
-		(property "Reference" "#PWR031"
+		(property "Reference" "#PWR061"
 			(at 86.36 113.03 0)
 			(hide yes)
@@
 			(project "pcb"
 				(path "/52b1b5de-c493-4cfe-b90b-d072cb2fb98d/9ecc0d26-f5db-4725-b97a-75ab22334c44"
-					(reference "#PWR031")
+					(reference "#PWR061")
 					(unit 1)
 				)
@@
 		(dnp no)
 		(fields_autoplaced yes)
-		(property "Reference" "#PWR034"
+		(property "Reference" "#PWR058"
 			(at 119.38 104.14 0)
 			(hide yes)
@@
 			(project "pcb"
 				(path "/52b1b5de-c493-4cfe-b90b-d072cb2fb98d/9ecc0d26-f5db-4725-b97a-75ab22334c44"
-					(reference "#PWR034")
+					(reference "#PWR058")
 					(unit 1)
 				)
@@
 		(in_pos_files yes)
 		(dnp no)
-		(property "Reference" "C28"
+		(property "Reference" "C38"
 			(at 173.99 99.0662 0)
 			(show_name no)
@@
 			(project "pcb"
 				(path "/52b1b5de-c493-4cfe-b90b-d072cb2fb98d/9ecc0d26-f5db-4725-b97a-75ab22334c44"
-					(reference "C28")
+					(reference "C38")
 					(unit 1)
 				)
@@
 		(in_pos_files yes)
 		(dnp no)
-		(property "Reference" "#PWR039"
+		(property "Reference" "#PWR055"
 			(at 243.84 43.18 0)
 			(hide yes)
@@
 			(project "pcb"
 				(path "/52b1b5de-c493-4cfe-b90b-d072cb2fb98d/9ecc0d26-f5db-4725-b97a-75ab22334c44"
-					(reference "#PWR039")
+					(reference "#PWR055")
 					(unit 1)
 				)
@@
 		(in_pos_files yes)
 		(dnp no)
-		(property "Reference" "C24"
+		(property "Reference" "C39"
 			(at 111.76 98.044 90)
 			(show_name no)
@@
 			(project "pcb"
 				(path "/52b1b5de-c493-4cfe-b90b-d072cb2fb98d/9ecc0d26-f5db-4725-b97a-75ab22334c44"
-					(reference "C24")
+					(reference "C39")
 					(unit 1)
 				)
@@
 		(in_pos_files yes)
 		(dnp no)
-		(property "Reference" "R7"
+		(property "Reference" "R11"
 			(at 118.11 83.058 90)
 			(show_name no)
@@
 			(project "pcb"
 				(path "/52b1b5de-c493-4cfe-b90b-d072cb2fb98d/9ecc0d26-f5db-4725-b97a-75ab22334c44"
-					(reference "R7")
+					(reference "R11")
 					(unit 1)
 				)
@@
 		(in_pos_files yes)
 		(dnp no)
-		(property "Reference" "R6"
+		(property "Reference" "R12"
 			(at 83.82 111.7599 0)
 			(show_name no)
@@
 			(project "pcb"
 				(path "/52b1b5de-c493-4cfe-b90b-d072cb2fb98d/9ecc0d26-f5db-4725-b97a-75ab22334c44"
-					(reference "R6")
+					(reference "R12")
 					(unit 1)
 				)
@@
 		(in_pos_files yes)
 		(dnp no)
-		(property "Reference" "C25"
+		(property "Reference" "C35"
 			(at 113.03 69.8562 0)
 			(show_name no)
@@
 			(project "pcb"
 				(path "/52b1b5de-c493-4cfe-b90b-d072cb2fb98d/9ecc0d26-f5db-4725-b97a-75ab22334c44"
-					(reference "C25")
-					(unit 1)
-				)
+					(reference "C35")
+					(unit 1)
+				)

Commit message: V2 fixup
Other:
- note added: "CPWG: 0.37mm Trace Width 0.22mm Gap ~49.9 ohm (D_{K} = 4.2 with 7628 prepreg) 7628 prepreg thickness is 0.2104 according to JLCPCB"
Changed lines of the file:
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@@
 		(title "Bluetooth")
 		(date "2026-10-09")
+		(rev "2")
 		(company "Dylan DiBeneditto")
 	)
@@
 		)
 	)
+	(text "CPWG:\n0.37mm Trace Width\n0.22mm Gap\n~49.9 ohm\n(D_{K} = 4.2 with 7628 prepreg)\n7628 prepreg thickness is 0.2104 according to JLCPCB"
+		(exclude_from_sim no)
+		(at 202.946 141.478 0)
+		(effects
+			(font
+				(size 1.27 1.27)
+			)
+			(justify left)
+		)
+	)
